File: hw/iomodul2.1/iomodul2.brd (EAGLE design)
At the start: 65 x 48 mm, 47 parts, among them IC1 MCP2551, IC3 STM32F042K, IC4 MCP1700T3302E/TT, IC5 DS8289, Q2 8MHz

Commit message: board version 3 begonnen
Parts:
- added LED3, LED4, LED5, LED6: (no value), led:CHIPLED_0805
- added Q1: (no value), crystal:HC49U-V
- added R11, R12, R13, R14: 68, schlager_passiv:R0805
- C1, C10, C11, C12, C13, C2, C25, C3, C4, C5, C6, C7, C8, C9: device schlager_passiv:C1206 -> schlager_passiv:C0805
- LED1, LED2: device led:CHIPLED_0603 -> led:CHIPLED_0805
- R1, R10, R2, R3, R4, R5, R6, R7, R8, R9: device schlager_passiv:R1206 -> schlager_passiv:R0805
- moved BR1 11.6 mm to (50.3, 41.7), turned to 180 degrees
- moved BR2 11.1 mm to (50.9, 5.94), turned to 180 degrees
- moved LED2 2.07 mm to (35.8, 28.0)
- moved C7 2.05 mm to (16.8, 24.9)
- moved C1 1.99 mm to (46.2, 6.99)
- moved LED1 1.81 mm to (35.8, 29.7)
- moved C2 1.80 mm to (15.0, 24.9)
- moved R5 1.55 mm to (30.8, 28.8)
- moved R4 1.55 mm to (37.0, 26.2)
- moved R3 1.42 mm to (30.8, 26.8)
- moved Q2 1.37 mm to (33.4, 18.4), turned to 270 degrees
- moved C4 1.02 mm to (37.0, 24.3)
- moved R6 0.89 mm to (37.0, 22.2)
- moved C6 0.63 mm to (32.0, 21.7)
- moved C10 0.51 mm to (32.0, 23.9)
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Connections:
- new net LED3_: IC3.14, R12.2, R13.2
- new net LED4_: IC3.15, R11.2, R14.2
- new net N$10: LED4.A, R12.1
- new net N$11: LED3.A, R11.1
- new net N$8: LED5.A, R13.1
- new net N$9: LED6.A, R14.1
- net +3V3: now also LED3.C, LED4.C, LED5.C, LED6.C
- net N$4: now also Q1.1
- net N$5: now also Q1.2
Routing:
- net +3V3: track 58.8 -> 102.9 mm, vias 2 -> 3
- net LED3_: track 0.00 -> 32.0 mm, vias 0 -> 2
- net CANL2: track 32.9 -> 63.9 mm, vias 1 -> 3
- net PE: track 0.00 -> 31.0 mm
- net CANH2: track 32.4 -> 59.7 mm, vias 1 -> 3
- net LED4_: track 0.00 -> 25.4 mm, vias 0 -> 2
- net CANL1: track 31.3 -> 56.4 mm, vias 1 -> 3
- net CANH1: track 29.9 -> 52.8 mm, vias 1 -> 2
- net +24V: track 136.5 -> 124.0 mm, vias 6 -> 4
- net N$2: track 13.7 -> 6.47 mm
- net N$5: track 7.67 -> 14.8 mm
- net N$4: track 12.7 -> 15.9 mm, vias 0 -> 1
- net N$1: track 0.00 -> 2.81 mm
- net N$11: track 0.00 -> 2.29 mm
- net N$9: track 0.00 -> 2.16 mm
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Other:
- board text added: "CAN-IOModul, 03'15 artwork by Sarah, Fablab KA Florolf, Entropia KA David Bauer, Fablab KA"
- board text removed: "CAN-IOModul, 10'14 artwork by Sarah, Fablab KA Florolf, Entropia KA"
