File: hw/iomodul2.1/iomodul2.sch (EAGLE design)
At the start: 47 parts, among them IC1 MCP2551, IC3 STM32F042K, IC4 MCP1700T3302E/TT, IC5 DS8289, Q2 8MHz

Commit message: board version 3 begonnen
Parts:
- added LED3, LED4, LED5, LED6: (no value), led:LEDCHIPLED_0805
- added Q1: (no value), crystal:CRYSTALHC49U-V
- added R11, R12, R13, R14: 68, schlager_passiv:R-EU_R0805
- C1, C10, C11, C12, C13, C2, C25, C3, C4, C5, C6, C7, C8, C9: device schlager_passiv:C-EUC1206 -> schlager_passiv:C-EUC0805
- LED1, LED2: device led:LEDCHIPLED_0603 -> led:LEDCHIPLED_0805
- R1, R10, R2, R3, R4, R5, R6, R7, R8, R9: device schlager_passiv:R-EU_R1206 -> schlager_passiv:R-EU_R0805
Connections:
- new net LED3_: IC3G$1.PB0/AIN8, R12.2, R13.2
- new net LED4_: IC3G$1.BP1/AIN9, R11.2, R14.2
- new net N$10: LED4.A, R12.1
- new net N$11: LED3.A, R11.1
- new net N$8: LED5.A, R13.1
- new net N$9: LED6.A, R14.1
- net +3V3: now also LED3.C, LED4.C, LED5.C, LED6.C
- net N$4: now also Q1.1
- net N$5: now also Q1.2
Other:
- moved on the sheet: BR1, BR2, C11, C4, C5, CON1G$1, CON2G$1, IC1, IC3, JP1, JP2, JP3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
