File: hw/canable mod/canable.brd (EAGLE design)
At the start: 19.1 x 45.1 mm, 25 parts, among them J2 USB-MICROB, U2 AP2202K-3.3TRG1, U3 MCP2551

Commit message: fixed board errors
Parts:
- moved C2 2.48 mm to (14.6, 20.2), turned to 90 degrees
- moved R3 0.16 mm to (12.9, 22.2)
Routing:
- net FGND: track 0.00 -> 22.6 mm
- net 3.3V: track 59.8 -> 56.1 mm
- net N$3: track 5.09 -> 7.78 mm, vias 0 -> 1
- net CANH: track 28.3 -> 30.9 mm
- net GND: vias 8 -> 11
