File: hw/Power-hub/power.brd (EAGLE design)
At the start: 100 x 100 mm, 71 parts, among them IC1 MCP2551, IC2 DS18B20, K1 615064243321, K2 61400826021, K3 61400826021, K4 615016240521

Commit message: neue Platinen
Parts:
- removed JP3: (no value), pinhead:2X09
- added C7: (no value), schlager_passiv:C0805
- added CON2: (no value), myconn:MEBP
- added IC3: MAX481CSA, maxim:SO08
- added JP4: (no value), pinhead:2X04
- added R28: (no value), schlager_passiv:R0805
- moved J8 20.0 mm to (94.8, 97.5)
- moved IC1 19.4 mm to (65.5, 75.1), turned to 180 degrees
- moved R17 14.0 mm to (88.9, 87.6)
- moved R1 13.1 mm to (67.5, 70.7), turned to 90 degrees
- moved R16 12.2 mm to (88.9, 89.7)
- moved C5 12.0 mm to (82.5, 97.8)
- moved C6 12.0 mm to (87.6, 97.8)
- moved Q1 12.0 mm to (85.1, 94.0)
- moved K4 8.98 mm to (86.4, 68.6)
- moved IC2 8.50 mm to (76.7, 94.8), turned to 270 degrees
- moved U$1 7.62 mm to (80.0, 85.1)
- moved JP1 6.35 mm to (68.8, 61.8)
- moved JP2 6.35 mm to (73.0, 61.9)
- moved C3 6.05 mm to (74.1, 75.9), turned to 270 degrees
- moved J5 5.08 mm to (85.1, 7.62)
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Connections:
- removed net 1W: IC2.2, JP3.15, U$2.12
- removed net DIG_O1: JP3.1, R13.2, R5.2, U$2.5
- removed net DIG_O2: JP3.3, R12.2, R14.2, U$2.6
- removed net DIG_O3: JP3.5, R11.2, R15.2, U$2.7
- removed net DIG_O4: JP3.7, R18.1, R22.2, U$2.8
- removed net DIG_O5: JP3.9, R19.1, R23.2, U$2.9
- removed net DIG_O6: JP3.11, R20.1, R24.2, U$2.10
- removed net DIG_O7: JP3.13, R21.1, R25.2, U$2.11
- removed net DIG_O8: JP3.4, R26.1, R27.2, U$2.19
- removed net N$16: U$2.2
- removed net N$19: JP3.8, U$2.17
- removed net N$25: JP3.6, U$2.18
- removed net N$8: U$2.1
- new net A0: JP4.2, U$2.17
- new net A1: IC3.2, IC3.3, U$2.18
- new net A2: R26.1, R27.2, U$2.19
- new net A6: JP4.6, U$2.A6
- new net A7: JP4.4, U$2.A7
- new net D2: R13.2, R5.2, U$2.5
- new net D3: R12.2, R14.2, U$2.6
- new net D4: R11.2, R15.2, U$2.7
- new net D5: R18.1, R22.2, U$2.8
- new net D6: R19.1, R23.2, U$2.9
- new net D7: R20.1, R24.2, U$2.10
- new net D8: R21.1, R25.2, U$2.11
- new net D9_1W: IC2.2, U$2.12
- new net N$3: CON2.T1, CON2.T2, R28.2
- new net RS485_A: CON2.1, CON2.7, IC3.6
- new net RS485_B: CON2.2, CON2.8, IC3.7
- new net RX: IC3.4, U$2.2
- new net SCL: JP4.5, U$2.A5
- new net SDA: JP4.3, U$2.A4
- new net TX: IC3.1, U$2.1
- net ANALOG_V24: no longer JP3.2
- net GND: now also C7.2, CON2.4, CON2.5, IC3.5, JP4.7, R28.1; no longer JP3.17
- net MISO: no longer JP3.12
- net MOSI: no longer JP3.14
- net P24P: now also CON2.3, CON2.6, JP4.8
- net P5V: now also C7.1, IC3.8, JP4.1; no longer JP3.18
- net SCK: no longer JP3.10
- net SS: no longer JP3.16
Routing:
- net DIG_O1: track 138.7 -> 0.00 mm, vias 1 -> 0
- net DIG_O7: track 124.5 -> 0.00 mm, vias 3 -> 0
- net DIG_O2: track 122.9 -> 0.00 mm, vias 2 -> 0
- net DIG_O6: track 110.6 -> 0.00 mm, vias 1 -> 0
- net DIG_O3: track 107.5 -> 0.00 mm
- net DIG_O5: track 105.7 -> 0.00 mm, vias 3 -> 0
- net DIG_O4: track 88.8 -> 0.00 mm, vias 1 -> 0
- net D2: track 0.00 -> 85.4 mm, vias 0 -> 1
- net D8: track 0.00 -> 70.7 mm
- net D3: track 0.00 -> 70.2 mm
- net D7: track 0.00 -> 58.7 mm
- net 1W: track 58.3 -> 0.00 mm, vias 3 -> 0
- net DIG_O8: track 55.4 -> 0.00 mm, vias 3 -> 0
- net D4: track 0.00 -> 50.9 mm
- net RX: track 0.00 -> 49.5 mm, vias 0 -> 1
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