File: hw/Power-hub/power.sch (EAGLE design)
At the start: 71 parts, among them IC1 MCP2551, IC2 DS18B20, K1 615064243321, K2 61400826021, K3 61400826021, K4 615016240521

Commit message: neue Platinen
Parts:
- removed JP3: (no value), pinhead:PINHD-2X9
- added C7: (no value), schlager_passiv:C-EUC0805
- added CON2: (no value), myconn:MEBP_8-8G
- added IC3: MAX481CSA, maxim:MAX481CSA
- added JP4: (no value), pinhead:PINHD-2X4
- added R28: (no value), schlager_passiv:R-EU_R0805
Connections:
- removed net 1W: IC2_1W.1W, JP3.15, U$2.*9
- removed net DIG_O1: JP3.1, R13.2, R5.2, U$2.2
- removed net DIG_O2: JP3.3, R12.2, R14.2, U$2.*3
- removed net DIG_O3: JP3.5, R11.2, R15.2, U$2.4
- removed net DIG_O4: JP3.7, R18.1, R22.2, U$2.*5
- removed net DIG_O5: JP3.9, R19.1, R23.2, U$2.*6
- removed net DIG_O6: JP3.11, R20.1, R24.2, U$2.7
- removed net DIG_O7: JP3.13, R21.1, R25.2, U$2.8
- removed net DIG_O8: JP3.4, R26.1, R27.2, U$2.A2
- removed net N$16: U$2.RXI
- removed net N$19: JP3.8, U$2.A0
- removed net N$25: JP3.6, U$2.A1
- removed net N$8: U$2.TXO
- new net A0: JP4.2, U$2.A0
- new net A1: IC3G$1.DE, IC3G$1.RE/, U$2.A1
- new net A2: R26.1, R27.2, U$2.A2
- new net A6: JP4.6, U$2.A6
- new net A7: JP4.4, U$2.A7
- new net D2: R13.2, R5.2, U$2.2
- new net D3: R12.2, R14.2, U$2.*3
- new net D4: R11.2, R15.2, U$2.4
- new net D5: R18.1, R22.2, U$2.*5
- new net D6: R19.1, R23.2, U$2.*6
- new net D7: R20.1, R24.2, U$2.7
- new net D8: R21.1, R25.2, U$2.8
- new net D9_1W: IC2_1W.1W, U$2.*9
- new net N$3: CON2G$2.FGND, R28.2
- new net RS485_A: CON2G$1.1, CON2G$1.7, IC3G$1.A
- new net RS485_B: CON2G$1.2, CON2G$1.8, IC3G$1.B
- new net RX: IC3G$1.DI, U$2.RXI
- new net SCL: JP4.5, U$2.A5
- new net SDA: JP4.3, U$2.A4
- new net TX: IC3G$1.RO, U$2.TXO
- net ANALOG_V24: no longer JP3.2
- net GND: now also C7.2, CON2G$1.4, CON2G$1.5, IC3P.GND, JP4.7, R28.1; no longer JP3.17
- net MISO: no longer JP3.12
- net MOSI: no longer JP3.14
- net P24P: now also CON2G$1.3, CON2G$1.6, JP4.8
- net P5V: now also C7.1, IC3P.VCC, JP4.1; no longer JP3.18
- net SCK: no longer JP3.10
- net SS: no longer JP3.16
Other:
- note added: "Spannungsmessung"
- note added: "ungenutze Pins"
