File: Gen2/Addon HR20/hr20.brd (EAGLE design)
At the start: 72.7 x 48 mm, 12 parts, among them SW1 430186043916, SW2 430186043916, SW3 430186043916

Commit message: ordner umsortiert und module weiter gemacht
Parts:
- moved SV1 2.54 mm to (64.8, 24.1)
Routing:
- net RX: track 30.1 -> 24.4 mm
- net TX: track 29.8 -> 27.3 mm
- net GND: track 162.9 -> 161.6 mm
Other:
- board size 72.7 x 48 mm -> 70 x 48 mm
Changed lines of the file:
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@@
 <wire x1="0" y1="0" x2="53.34" y2="0" width="0" layer="20"/>
 <wire x1="53.34" y1="0" x2="53.34" y2="6.35" width="0" layer="20"/>
-<wire x1="53.34" y1="6.35" x2="72.7" y2="6.35" width="0" layer="20"/>
-<wire x1="72.7" y1="6.35" x2="72.7" y2="41.91" width="0" layer="20"/>
-<wire x1="72.7" y1="41.91" x2="53.34" y2="41.91" width="0" layer="20"/>
+<wire x1="53.34" y1="6.35" x2="70" y2="6.35" width="0" layer="20"/>
+<wire x1="70" y1="6.35" x2="70" y2="41.91" width="0" layer="20"/>
+<wire x1="70" y1="41.91" x2="53.34" y2="41.91" width="0" layer="20"/>
 <wire x1="53.34" y1="41.91" x2="53.34" y2="48" width="0" layer="20"/>
 <wire x1="53.34" y1="48" x2="0" y2="48" width="0" layer="20"/>
@@
 <element name="JP5" library="pinhead" package="1X08" value="" x="21.59" y="7.62"/>
 <element name="JP6" library="pinhead" package="1X10" value="" x="13.97" y="40.64"/>
-<element name="SV1" library="X_Pfostenstecker" package="ML10" value="" x="67.31" y="24.13" rot="R90">
-<attribute name="OC_NEWARK" value="unknown" x="20.32" y="24.13" size="1.778" layer="27" font="vector" rot="R90" display="off"/>
-<attribute name="MPN" value="" x="20.32" y="24.13" size="1.778" layer="27" font="vector" rot="R90" display="off"/>
-<attribute name="MF" value="" x="20.32" y="24.13" size="1.778" layer="27" font="vector" rot="R90" display="off"/>
-<attribute name="OC_FARNELL" value="unknown" x="20.32" y="24.13" size="1.778" layer="27" font="vector" rot="R90" display="off"/>
+<element name="SV1" library="X_Pfostenstecker" package="ML10" value="" x="64.77" y="24.13" rot="R90">
+<attribute name="OC_NEWARK" value="unknown" x="17.78" y="24.13" size="1.778" layer="27" font="vector" rot="R90" display="off"/>
+<attribute name="MPN" value="" x="17.78" y="24.13" size="1.778" layer="27" font="vector" rot="R90" display="off"/>
+<attribute name="MF" value="" x="17.78" y="24.13" size="1.778" layer="27" font="vector" rot="R90" display="off"/>
+<attribute name="OC_FARNELL" value="unknown" x="17.78" y="24.13" size="1.778" layer="27" font="vector" rot="R90" display="off"/>
 </element>
 <element name="U$2" library="schlager_modules" package="1.44-128X128" value="1.44-128X128" x="0.3175" y="1.74625"/>
@@
 <wire x1="17.78" y1="43.18" x2="17.78" y2="40.64" width="0.4064" layer="16"/>
 <wire x1="57.15" y1="24.13" x2="57.15" y2="33.02" width="0.4064" layer="16"/>
-<wire x1="66.04" y1="29.21" x2="66.04" y2="30.48" width="0.4064" layer="16"/>
-<wire x1="66.04" y1="30.48" x2="58.42" y2="38.1" width="0.4064" layer="16"/>
+<wire x1="63.5" y1="29.21" x2="63.5" y2="31.75" width="0.4064" layer="16"/>
+<wire x1="63.5" y1="31.75" x2="58.42" y2="38.1" width="0.4064" layer="16"/>
 <wire x1="58.42" y1="38.1" x2="50.8" y2="38.1" width="0.4064" layer="16"/>
 <wire x1="50.8" y1="38.1" x2="49.53" y2="39.37" width="0.4064" layer="16"/>
@@
 <wire x1="41.91" y1="15.24" x2="41.91" y2="19.9" width="0.4064" layer="16"/>
 <wire x1="41.91" y1="19.9" x2="43.89" y2="21.88" width="0.4064" layer="16"/>
-<wire x1="68.58" y1="29.21" x2="67.31" y2="27.94" width="0.4064" layer="16"/>
+<wire x1="66.04" y1="29.21" x2="67.31" y2="27.94" width="0.4064" layer="16"/>
 <wire x1="67.31" y1="27.94" x2="67.31" y2="16.51" width="0.4064" layer="16"/>
 <wire x1="67.31" y1="16.51" x2="62.23" y2="11.43" width="0.4064" layer="16"/>
@@
 <wire x1="59.69" y1="33.02" x2="59.69" y2="25.4" width="0.4064" layer="16"/>
 <wire x1="59.69" y1="25.4" x2="60.96" y2="24.13" width="0.4064" layer="16"/>
-<wire x1="60.96" y1="24.13" x2="66.04" y2="24.13" width="0.4064" layer="16"/>
+<wire x1="60.96" y1="24.13" x2="63.5" y2="24.13" width="0.4064" layer="16"/>
 <wire x1="52.07" y1="35.56" x2="48.26" y2="39.37" width="0.4064" layer="16"/>
 <wire x1="48.26" y1="39.37" x2="48.26" y2="40.64" width="0.4064" layer="16"/>
@@
 <contactref element="JP1" pad="1"/>
 <contactref element="SV1" pad="7"/>
-<wire x1="50.8" y1="40.64" x2="62.23" y2="40.64" width="0.4064" layer="16"/>
-<wire x1="62.23" y1="40.64" x2="71.12" y2="31.75" width="0.4064" layer="16"/>
-<wire x1="71.12" y1="31.75" x2="71.12" y2="29.21" width="0.4064" layer="16"/>
-<wire x1="71.12" y1="29.21" x2="68.58" y2="26.67" width="0.4064" layer="16"/>
+<wire x1="50.8" y1="40.64" x2="58.42" y2="40.64" width="0.4064" layer="16"/>
+<wire x1="58.42" y1="40.64" x2="64.77" y2="33.02" width="0.4064" layer="16"/>
+<wire x1="64.77" y1="33.02" x2="64.77" y2="27.94" width="0.4064" layer="16"/>
+<wire x1="64.77" y1="27.94" x2="66.04" y2="26.67" width="0.4064" layer="16"/>
 </signal>
 <signal name="D10_SS">
