File: Nodes Gen2/Addon HR20/hr20.sch (EAGLE design)
At the start: 12 parts, among them SW1 430186043916, SW2 430186043916, SW3 430186043916

Commit message: gen 2 dev + bom
Parts:
- removed JP1, JP5: (no value), pinhead:PINHD-1X8
- removed JP4: (no value), pinhead:PINHD-1X6
- removed JP6: (no value), pinhead:PINHD-1X10
- added JP2, JP3, JP8: (no value), pinhead:PINHD-1X8
- added JP7: (no value), pinhead:PINHD-2X4
Connections:
- removed net A4_SDA1: JP6.9
- removed net A4_SDA2: JP4.5
- removed net A5_SCL1: JP6.10
- removed net A5_SCL2: JP4.6
- removed net A6: JP5.8
- removed net A7: JP5.7
- removed net AREF: JP6.8
- removed net D8: JP6.1
- removed net D9: JP6.2, U$2.P$5
- new net A4_SDA: JP3.5
- new net A5_SCL: JP3.6
- new net D8_SS: JP8.1, U$2.P$3
- new net D9_SS: JP8.2
- new net RESERVE2: JP8.8
- net A0: now also JP3.1; no longer JP4.1
- net A1: now also JP3.2; no longer JP4.2
- net A2: now also JP3.3; no longer JP4.3
- net A3_V24: now also JP3.4; no longer JP4.4
- net D10_SS: now also JP8.3; no longer JP6.3, U$2.P$3
- net D11_MOSI: now also JP8.4; no longer JP6.4
- net D12_MISO: now also JP8.5; no longer JP6.5
- net D13_SCK: now also JP8.6; no longer JP6.6
- net D2: now also JP2.3; no longer JP1.3
- net D3: now also JP2.4; no longer JP1.4
- net D4: now also JP2.5; no longer JP1.5
- net D5: now also JP2.6; no longer JP1.6
- net D6: now also JP2.7; no longer JP1.7
- net D7: now also JP2.8; no longer JP1.8
- net GND: now also JP7.3, JP7.4; no longer JP5.3, JP5.4, JP6.7
- net P24P: now also JP7.7, JP7.8; no longer JP5.1, JP5.2
- net P5V: now also JP7.1, JP7.2; no longer JP5.5, JP5.6
- net RESET: now also JP8.7
- net RX: now also JP2.1; no longer JP1.1
- net TX: now also JP2.2; no longer JP1.2
