File: Nodes Gen2/Addon RGBW/rgbw2.sch (EAGLE design)
At the start: 33 parts, among them Q1 BUZ11SD, Q2 BUZ11SD, Q3 BUZ11SD, Q4 BUZ11SD, Q5 BUZ11SD, Q6 BUZ11SD, Q7 BUZ11SD, Q8 BUZ11SD

Commit message: gen 2 dev + bom
Parts:
- removed JP1, JP5: (no value), pinhead:PINHD-1X8
- removed JP4: (no value), pinhead:PINHD-1X6
- removed JP6: (no value), pinhead:PINHD-1X10
- removed Q8: BUZ11SD, transistor-fet:BUZ11SD
- added JP3, JP8, JP9: (no value), pinhead:PINHD-1X8
- added JP7: (no value), pinhead:PINHD-2X4
- added Q9: MOSFET-NCHANNELFDD8780, SparkFun-DiscreteSemi:MOSFET-NCHANNELFDD8780
- added R10, R11, R12, R13, R14, R9: (no value), schlager_passiv:R-EU_R0805
- added SJ10, SJ11, SJ12, SJ13, SJ14, SJ6: (no value), jumper:SJN
- Q1, Q2, Q3, Q4, Q5, Q6, Q7: value BUZ11SD -> MOSFET-NCHANNELFDD8780; device transistor-fet:BUZ11SD -> SparkFun-DiscreteSemi:MOSFET-NCHANNELFDD8780
- SJ1, SJ2, SJ3, SJ4, SJ5, SJ7, SJ8, SJ9: device jumper:SJ -> jumper:SJN
Connections:
- removed net A3_SCL2: JP4.4
- removed net A4_SDA2: JP4.5
- removed net A5: JP4.6
- removed net AREF: JP6.8
- new net A3_V24: JP8.4
- new net N$1: R9.1, SJ6.2, U1.A0
- new net N$10: R10.1, SJ10.2, U1.A1
- new net N$11: R11.1, SJ11.2, U1.A2
- new net N$12: R12.1, SJ12.2, U1.A3
- new net N$13: R13.1, SJ13.2, U1.A4
- new net N$14: R14.1, SJ14.2, U1.A5
- new net RESERVE: JP9.7
- new net RESERVE2: JP9.8
- net A0: now also JP8.1; no longer JP4.1
- net A1: now also JP8.2; no longer JP4.2
- net A2: now also JP8.3; no longer JP4.3
- net A4_SDA: now also JP8.5, U1.SDA; no longer JP6.9
- net A5_SCL: now also JP8.6, U1.SCL; no longer JP6.10
- net A6: now also JP8.7; no longer JP5.8
- net A7: now also JP8.8; no longer JP5.7
- net D10_SS: now also JP9.3; no longer JP6.3
- net D11_MOSI: now also JP9.4; no longer JP6.4
- net D12_MISO: now also JP9.5; no longer JP6.5
- net D13_SCK: now also JP9.6; no longer JP6.6
- net D2: now also JP3.3; no longer JP1.3
- net D3: now also JP3.4; no longer JP1.4
- net D4: now also JP3.5; no longer JP1.5
- net D5: now also JP3.6; no longer JP1.6
- net D6: now also JP3.7; no longer JP1.7
- net D7: now also JP3.8; no longer JP1.8
- net D8: now also JP9.1; no longer JP6.1
- net D9: now also JP9.2; no longer JP6.2
- net GND: now also JP7.3, JP7.4, Q9.S, SJ10.1, SJ11.1, SJ12.1, SJ13.1, SJ14.1, SJ6.1, U1.GND; no longer JP5.3, JP5.4, JP6.7, Q8.S
- net LED0: now also Q9.G; no longer Q2.G
- net LED1: now also Q1.G; no longer Q3.G
- net LED2: now also Q2.G; no longer Q4.G
- net LED3: now also Q3.G; no longer Q5.G
- net LED4: now also Q7.G; no longer Q1.G
- net LED6: now also Q5.G; no longer Q7.G
- net LED7: now also Q4.G; no longer Q8.G
- net N$2: now also Q9.D; no longer Q2.D
- net N$3: now also Q1.D; no longer Q3.D
- net N$4: now also Q5.D; no longer Q7.D
- net N$5: now also Q2.D; no longer Q4.D
- net N$6: now also Q3.D; no longer Q5.D
- net N$7: now also Q4.D; no longer Q8.D
- net N$8: now also Q7.D; no longer Q1.D
- net P24P: now also JP7.7, JP7.8; no longer JP5.1, JP5.2
- net P24X: now also JP7.5, JP7.6
- net P5V: now also JP7.1, JP7.2, R10.2, R11.2, R12.2, R13.2, R14.2, R9.2, U1.VDD; no longer JP5.5, JP5.6
- net RX: now also JP3.1; no longer JP1.1
- net TX: now also JP3.2; no longer JP1.2
