File: Nodes Gen2/Basis/basis.brd (EAGLE design)
At the start: 100 x 48 mm, 27 parts, among them IC1 DS1820TO92, IC2 MCP2551, IC3 MAX481CSA, K4 615016240521

Commit message: gen 2 dev + bom
Parts:
- added C3: (no value), schlager_passiv:C0805
- added JP7: (no value), pinhead:2X04
- C7, C8: value (none) -> 100UF; device schlager_passiv:E5-10,5 -> PASSIV_Panasonic-EEEFK_EEEFP:CAPAE830X1050N
- JP4: device pinhead:1X06 -> pinhead:1X08
- JP6: device pinhead:1X10 -> pinhead:1X03/90
- moved JP4 48.8 mm to (47.0, 38.1), turned to 270 degrees
- moved JP5 43.1 mm to (92.7, 38.1), turned to 270 degrees
- moved C1 42.3 mm to (86.4, 45.2), turned to 0 degrees
- moved JP6 40.0 mm to (55.9, 0.64), turned to 180 degrees
- moved C6 32.7 mm to (63.3, 43.8), turned to 90 degrees
- moved JP1 32.1 mm to (92.7, 10.2), turned to 90 degrees
- moved R3 29.7 mm to (57.1, 37.6), turned to 0 degrees
- moved IC2 29.0 mm to (59.7, 39.4)
- moved Q1 26.5 mm to (67.3, 40.6), turned to 90 degrees
- moved C5 26.1 mm to (63.3, 37.6), turned to 270 degrees
- moved U$3 25.2 mm to (77.5, 40.6), turned to 0 degrees
- moved IC3 12.7 mm to (57.1, 31.8), turned to 90 degrees
- moved U$1 10.6 mm to (76.5, 16.5), turned to 180 degrees
- moved C2 5.71 mm to (57.1, 27.9), turned to 0 degrees
- moved C8 1.00 mm to (9.84, 40.5)
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Connections:
- net A3_V24 renamed A3
- removed net A5: JP4.6
- removed net AREF: JP6.8
- removed net D7: JP1.8, U$1.10
- removed net D8: IC1.2, JP6.1, R1.1, U$1.11
- removed net D9: IC3.2, IC3.3, JP6.2, U$1.12
- new net 1W: IC1.2, JP1.8, JP6.2, R1.1, U$1.10
- new net D8_SS: JP5.1, U$1.11
- new net D9_SS: IC3.2, IC3.3, JP5.2, U$1.12
- new net RESERVE: JP5.7
- new net RESERVE2: JP5.8
- net A4_SDA: no longer JP6.9
- net A5_SCL: now also JP4.6; no longer JP6.10
- net A6: no longer JP5.8
- net A7: no longer JP5.7
- net D10_SS: now also JP5.3; no longer JP6.3
- net D11_MOSI: now also JP5.4; no longer JP6.4
- net D12_MISO: now also JP5.5; no longer JP6.5
- net D13_SCK: now also JP5.6; no longer JP6.6
- net GND: now also C3.2, C7.2, C8.2, IC2.2, JP6.3, JP7.3, JP7.4; no longer C7.-, C8.-, JP5.3, JP5.4, JP6.7
- net P24P: now also C7.1, JP7.7, JP7.8; no longer C7.+, JP5.1, JP5.2
- net P5V: now also C3.1, C8.1, IC2.3, JP6.1, JP7.1, JP7.2; no longer C8.+, JP5.5, JP5.6
Routing:
- net 1W: track 0.00 -> 129.9 mm, vias 0 -> 9
- net D8: track 64.4 -> 0.00 mm, vias 1 -> 0
- net D9_SS: track 0.00 -> 56.8 mm, vias 0 -> 3
- net CANH: track 4.77 -> 46.2 mm, vias 0 -> 5
- net A1: track 9.34 -> 47.3 mm, vias 0 -> 2
- net A3: track 9.34 -> 47.3 mm, vias 0 -> 2
- net A2: track 9.34 -> 47.3 mm, vias 0 -> 2
- net A0: track 9.34 -> 47.3 mm, vias 0 -> 2
- net D9: track 34.1 -> 0.00 mm, vias 2 -> 0
- net GND: track 33.2 -> 4.01 mm, vias 6 -> 1
- net CANL: track 9.85 -> 38.8 mm, vias 0 -> 5
- net A6: track 28.6 -> 0.00 mm
- net D8_SS: track 0.00 -> 26.4 mm, vias 0 -> 2
- net A7: track 21.8 -> 0.00 mm
- net CANRX: track 5.60 -> 19.0 mm, vias 0 -> 4
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- added copper zone on layer 1, net GND
- added copper zone on layer 16, net P24P
- added copper zone on layer 16, net P5V
- removed copper zone on layer 16, net GND
- removed copper zone on layer 1, net N$1
- removed copper zone on layer 1, net P24P
- removed copper zone on layer 1, net P5V
Other:
- board text removed: "ESP8255-01"
- board text removed: "i2c"
