File: Nodes Gen2/Basis/basis.sch (EAGLE design)
At the start: 27 parts, among them IC1 DS1820TO92, IC2 MCP2551, IC3 MAX481CSA, K4 615016240521

Commit message: gen 2 dev + bom
Parts:
- added C3: (no value), schlager_passiv:C-EUC0805
- added JP7: (no value), pinhead:PINHD-2X4
- C7, C8: value (none) -> 100UF; device schlager_passiv:CPOL-EUE5-10.5 -> PASSIV_Panasonic-EEEFK_EEEFP:EEE-FK1V101P-CASE-F
- JP4: device pinhead:PINHD-1X6 -> pinhead:PINHD-1X8
- JP6: device pinhead:PINHD-1X10 -> pinhead:PINHD-1X3/90
Connections:
- net A3_V24 renamed A3
- removed net A5: JP4.6
- removed net AREF: JP6.8
- removed net D7: JP1.8, U$1.7
- removed net D8: IC1.DQ, JP6.1, R1.1, U$1.8
- removed net D9: IC3G$1.DE, IC3G$1.RE/, JP6.2, U$1.*9
- new net 1W: IC1.DQ, JP1.8, JP6.2, R1.1, U$1.7
- new net D8_SS: JP5.1, U$1.8
- new net D9_SS: IC3G$1.DE, IC3G$1.RE/, JP5.2, U$1.*9
- new net RESERVE: JP5.7
- new net RESERVE2: JP5.8
- net A4_SDA: no longer JP6.9
- net A5_SCL: now also JP4.6; no longer JP6.10
- net A6: no longer JP5.8
- net A7: no longer JP5.7
- net D10_SS: now also JP5.3; no longer JP6.3
- net D11_MOSI: now also JP5.4; no longer JP6.4
- net D12_MISO: now also JP5.5; no longer JP6.5
- net D13_SCK: now also JP5.6; no longer JP6.6
- net GND: now also C3.2, C7.2, C8.2, IC2G$2.GND, JP6.3, JP7.3, JP7.4; no longer C7.-, C8.-, JP5.3, JP5.4, JP6.7
- net P24P: now also C7.1, JP7.7, JP7.8; no longer C7.+, JP5.1, JP5.2
- net P5V: now also C3.1, C8.1, IC2G$2.VCC, JP6.1, JP7.1, JP7.2; no longer C8.+, JP5.5, JP5.6
Other:
- moved on the sheet: JP5
