File: Nodes Gen2/Addon GPIO/addonv2.brd (EAGLE design)
At the start: 60 x 48 mm, 55 parts

Commit message: so much...
Parts:
- removed JP16: (no value), pinhead:1X04/90
- added JP5: (no value), pinhead:1X04/90
- added U$2: (no value), debauer_special:KALT!ELEKTRONIK
- added U$3, U$4, U$5, U$7: (no value), debauer_special:PASSMARK
- added U$8: (no value), debauer_special:LABNET
- R1, R17, R18, R19, R2, R20, R21, R22, R23, R24, R25, R26, R27, R28, R29, R3, R30, R31, R4, R5, R6, R7, R8: device rcl:R0805 -> debauer_passiv:R0603
- moved R22 0.16 mm to (88.9, 39.4)
Connections:
- net A4_SDA: now also JP5.2; no longer JP16.3
- net A5_SCL: now also JP5.3; no longer JP16.4
- net GND: now also JP5.1; no longer JP16.2
- net P5V: now also JP5.4; no longer JP16.1
Routing:
- net P5V: track 15.2 -> 46.3 mm, vias 6 -> 8
- net A4_SDA: track 110.0 -> 113.3 mm
- net P24P: track 0.00 -> 2.54 mm
- net A5_SCL: track 99.6 -> 101.8 mm
- net A2: track 55.1 -> 56.9 mm
- net A0: track 66.3 -> 65.6 mm
Other:
- board text added: "0"
- board text added: "5V"
- board text added: "A0"
- board text added: "A1"
- board text added: "A1 A0"
- board text added: "A2"
- board text added: "A3"
- board text added: "A3 A2"
- board text added: "A7 A6"
- board text added: "ADS1115"
- board text added: "Analog In"
- board text added: "Design: David Bauer"
- board text added: "GND"
- board text added: "GPIO1.0"
- board text added: "MCP23S17"
- board text added: "RELAI"
- board text added: "SCL"
- board text added: "SDA"
- board text added: "Status LEDs"
- board text added: "i2c"
- board text added: "www.debauer.net"
- board text added: "www.fablab-karlsruhe.de"
- board text added: "www.kalt-elektronik.de"
- board text removed: "10"
- board text removed: "11"
- board text removed: "12"
- board text removed: "13"
- board text removed: "14"
- board text removed: "15"
- board text removed: "16"
- board text removed: "8"
- board text removed: "9"
