File: Nodes Gen2/Addon LCD_LED/addonv2.sch (EAGLE design)
At the start: 51 parts, among them SW1 430152043826, SW2 430152043826, SW3 430152043826

Commit message: so much...
Connections:
- new net N$33: U$1.INTA
- new net N$34: U$1.INTB
Changed lines of the file:
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@@
 <wire x1="177.8" y1="152.4" x2="182.88" y2="152.4" width="0.1524" layer="91"/>
 <junction x="177.8" y="152.4"/>
+<label x="185.42" y="152.4" size="1.778" layer="95"/>
 </segment>
 </net>
@@
 <pinref part="SW2" gate="G$1" pin="3"/>
 <junction x="157.734" y="137.16"/>
+<label x="185.42" y="137.16" size="1.778" layer="95"/>
 </segment>
 </net>
@@
 <wire x1="182.88" y1="121.92" x2="172.72" y2="121.92" width="0.1524" layer="91"/>
 <junction x="172.72" y="121.92"/>
+<label x="185.42" y="121.92" size="1.778" layer="95"/>
 </segment>
 </net>
@@
 </segment>
 </net>
+<net name="N$33" class="0">
+<segment>
+<pinref part="U$1" gate="A" pin="INTA"/>
+<wire x1="203.2" y1="213.36" x2="208.28" y2="213.36" width="0.1524" layer="91"/>
+</segment>
+</net>
+<net name="N$34" class="0">
+<segment>
+<pinref part="U$1" gate="A" pin="INTB"/>
+<wire x1="208.28" y1="210.82" x2="203.2" y2="210.82" width="0.1524" layer="91"/>
+</segment>
+</net>
