File: Nodes Gen2/Addon Motor/motor.brd (EAGLE design)
At the start: 59.4 x 48 mm, 25 parts

Commit message: gen 2 dev + bom
Parts:
- removed J1: (no value), Eagle_TERMINAL_BLOCKS_rev16a:691312510004
- removed JP5: (no value), pinhead:1X08
- removed JP6: (no value), pinhead:1X10
- added JP10, JP13, JP14: (no value), pinhead:1X08
- added JP12: (no value), pinhead:2X04
- J2: device Eagle_TERMINAL_BLOCKS_rev16a:691312510004 -> Eagle_TERMINAL_BLOCKS_rev16a:691322310002
- JP1: device pinhead:1X08 -> pinhead:1X04/90
- JP4: device pinhead:1X06 -> pinhead:1X04/90
- moved J2 72.4 mm to (0.00, -24.1)
- moved U$2 68.6 mm to (82.5, 25.4)
- moved R2 67.7 mm to (88.9, 34.3), turned to 90 degrees
- moved R3 65.0 mm to (86.4, 34.3), turned to 270 degrees
- moved R7 53.5 mm to (86.4, 38.1), turned to 90 degrees
- moved R8 52.5 mm to (88.9, 38.1), turned to 90 degrees
- moved J3 51.4 mm to (59.1, 2.54)
- moved JP1 49.7 mm to (68.6, -1.27)
- moved JP4 48.7 mm to (69.2, 49.5)
- moved C1 44.0 mm to (79.2, 36.8), turned to 0 degrees
- moved C2 43.3 mm to (54.9, 37.0)
- moved R5 42.9 mm to (82.1, 8.57), turned to 270 degrees
- moved JP2 41.9 mm to (68.6, 24.1)
- moved JP11 41.8 mm to (78.7, 49.5)
- moved R6 41.6 mm to (84.3, 8.57), turned to 270 degrees
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Connections:
- removed net 1A1: J1.4, U$2.1A
- removed net 1A2: J2.4, U$1.1A
- removed net 1B1: J1.3, U$2.1B
- removed net 1B2: J2.3, U$1.1B
- removed net 2A1: J1.2, U$2.2A
- removed net 2A2: J2.2, U$1.2A
- removed net 2B1: J1.1, U$2.2B
- removed net 2B2: J2.1, U$1.2B
- removed net A3_SCL2: JP4.4
- removed net A4_SDA2: JP4.5
- removed net A6: JP5.8
- removed net A7: JP5.7
- removed net AREF: JP6.8
- new net N$11: JP1.4, U$2.1A
- new net N$12: JP1.3, U$2.1B
- new net N$13: JP1.2, U$2.2A
- new net N$14: JP1.1, U$2.2B
- new net N$15: JP4.1, U$1.2B
- new net N$16: JP4.2, U$1.2A
- new net N$17: JP4.3, U$1.1B
- new net N$18: JP4.4, U$1.1A
- new net RESERVE: JP14.7
- new net RESERVE2: JP14.8
- net A4_SDA: now also JP13.5; no longer JP6.9
- net A5_SCL: now also JP13.6; no longer JP6.10
- net D10_SS: now also JP14.3; no longer JP6.3
- net D11_MOSI: now also JP14.4; no longer JP6.4
- net D12_MISO: now also JP14.5; no longer JP6.5
- net D13_SCK: now also JP14.6; no longer JP6.6
- net D2: now also JP10.3; no longer JP1.3
- net D3: now also JP10.4; no longer JP1.4
- net D4: now also JP10.5; no longer JP1.5
- net D5: now also JP10.6; no longer JP1.6
- net END1: now also JP10.7; no longer JP1.7
- net END2: now also JP10.8; no longer JP1.8
- net END3: now also JP13.1; no longer JP4.1
- net END4: now also JP13.2; no longer JP4.2
- net GND: now also JP12.3, JP12.4; no longer JP5.3, JP5.4, JP6.7
- net P24P: now also JP12.7, JP12.8; no longer JP5.1, JP5.2
- net P5V: now also JP12.1, JP12.2; no longer JP5.5, JP5.6
- net RX: now also JP10.1; no longer JP1.1
- net SERVO1: now also JP14.1; no longer JP6.1
- net SERVO2: now also JP14.2; no longer JP6.2
- net SERVO3: now also JP13.3; no longer JP4.3
- net SERVO4: now also JP13.4; no longer JP4.6
- net TX: now also JP10.2; no longer JP1.2
Routing:
- net N$18: track 0.00 -> 43.8 mm
- net 1A1: track 43.6 -> 0.00 mm, vias 2 -> 0
- net 1A2: track 43.3 -> 0.00 mm, vias 1 -> 0
- net END1: track 5.18 -> 47.3 mm, vias 0 -> 1
- net 1B1: track 41.3 -> 0.00 mm
- net END2: track 12.1 -> 53.2 mm, vias 0 -> 3
- net N$17: track 0.00 -> 39.5 mm
- net N$16: track 0.00 -> 35.9 mm
- net SERVO4: track 6.88 -> 40.7 mm, vias 0 -> 2
- net 1B2: track 32.9 -> 0.00 mm
- net N$14: track 0.00 -> 32.5 mm
- net N$15: track 0.00 -> 31.9 mm
- net END3: track 7.14 -> 39.0 mm, vias 0 -> 3
- net N$13: track 0.00 -> 30.5 mm
- net 2A1: track 30.4 -> 0.00 mm, vias 1 -> 0
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Other:
- board text removed: "+"
- board text removed: "-"
- board text removed: "ENDSTOP"
- board text removed: "Servo"
- board text removed: "Stepper 1"
- board text removed: "Stepper 2"

Commit message: so much...
Parts:
- removed J2: (no value), Eagle_TERMINAL_BLOCKS_rev16a:691322310002
- added U$3, U$8: (no value), debauer_special:PASSMARK
- added U$4: (no value), debauer_special:SNOW
- added U$6: (no value), debauer_special:KALT!ELEKTRONIK
- added U$7: (no value), debauer_special:LABNET
- moved C1 0.48 mm to (78.7, 36.8)
- moved R5 0.32 mm to (81.8, 8.57)
- moved R6 0.32 mm to (84.6, 8.57)
Connections:
- new net A6: JP13.7
- new net A7: JP13.8
Routing:
- net P5V: track 15.0 -> 15.5 mm
Other:
- board text added: "4"
- board text added: "Design: David Bauer"
- board text added: "END 1/2"
- board text added: "END 3/4"
- board text added: "GNDM"
- board text added: "MOT1"
- board text added: "MOT2"
- board text added: "MOTOR1.0"
- board text added: "PWR IN"
- board text added: "PWRM"
- board text added: "STEP 1/2"
- board text added: "STEP 3/4"
- board text added: "STEPSTICK"
- board text added: "www.fablab-karlsruhe.de"
- board text added: "www.kalt-elektronik.de"
- board text removed: "FabLab KA"
- board text removed: "Motor Addon by debauer"
