File: Nodes Gen2/Basis KFZ/basis.brd (EAGLE design)
At the start: 100 x 48 mm, 36 parts, among them IC1 DS1820TO92, IC2 MCP2551, IC3 MAX481CSA, K4 615016240521, U1 AT24C64CN-SH-B

Commit message: so much...
Parts:
- removed U$5, U$7, U$8: (no value), debauer_special:LABNET
- moved U$2 22.8 mm to (76.4, 12.5), turned to 90 degrees
- moved C8 2.40 mm to (9.84, 40.5)
- moved C4 2.38 mm to (64.3, 19.5)
Routing:
- net P5V: track 33.2 -> 30.6 mm
Other:
- board text removed: "1Wire"
- board text removed: "5"
- board text removed: "5V 5A"
- board text removed: "CAN"
- board text removed: "D"
- board text removed: "Design: David Bauer"
- board text removed: "G"
- board text removed: "MCP2515"
- board text removed: "MCP2551"
- board text removed: "PWR"
- board text removed: "RS485"
- board text removed: "www.debauer.net"
- board text removed: "www.fablab-karlsruhe.de"
