File: Nodes Gen2/Basis KFZ/basis.sch (EAGLE design)
At the start: 31 parts, among them IC1 DS1820TO92, IC2 MCP2551, IC3 MAX481CSA, K4 615016240521, U1 AT24C64CN-SH-B

Commit message: so much...
Parts:
- removed C1, C2: 100n, schlager_passiv:C-EUC0805
- removed CON1: (no value), myconn:MEBP_8-8G
- removed IC3: MAX481CSA, maxim:MAX481CSA
- removed JP3: (no value), jumper:JP2E
- removed R2: 1M, schlager_passiv:R-EU_R0805
- added J1: (no value), Wuerth_TERMINAL_BLOCKS_rev16a:691317510003
- added K1: G5LE, relay:G5LE
- added U$5: ES2D, debauer_dioden:ES2D
- added U2: LM1117MP-ADJ, debauer_reg:LM1117MP-ADJ
- JP2: device jumper:JP2E -> pinhead:PINHD-2X4
Connections:
- removed net RS485_A: CON1G$1.1, CON1G$1.7, IC3G$1.A
- removed net RS485_B: CON1G$1.2, CON1G$1.8, IC3G$1.B
- new net GND24X: C3.2, IC2G$2.GND, K4.A4, K4.A5, K4.B4, K4.B5, R3.2, U2.ADJ/GND
- new net P24X: K4.A3, K4.A6, K4.B3, K4.B6, U2.IN
- new net P5X: C3.1, IC2G$2.VCC, U2.OUT, U2.VOUT
- new net ZUEND_KFZ: J1.2, K11.1, U$5.C
- net CANH: now also JP2.1, JP2.3; no longer JP3.2
- net CANH1: now also JP2.2; no longer JP3.3
- net CANH2: now also JP2.4; no longer JP3.1
- net CANL: now also JP2.5, JP2.7; no longer JP2.2
- net CANL1: now also JP2.6; no longer JP2.3
- net CANL2: now also JP2.8; no longer JP2.1
- net D9_SS: no longer IC3G$1.DE, IC3G$1.RE/
- net GND: now also J1.1, K11.2, U$5.A; no longer C1.2, C2.2, C3.2, CON1G$1.4, CON1G$1.5, IC2G$2.GND, IC3P.GND, K4.A4, K4.A5, K4.B4, K4.B5, R2.1, R3.2
- net N$3: now also J1.3, K12.S; no longer CON1G$2.FGND, R2.2
- net P24P: now also K12.P; no longer CON1G$1.3, CON1G$1.6, K4.A3, K4.A6, K4.B3, K4.B6
- net P5V: no longer C1.1, C2.1, C3.1, IC2G$2.VCC, IC3P.VCC
- net RX: no longer IC3G$1.DI
- net TX: no longer IC3G$1.RO
