File: Nodes Gen2/Power-hub/power.brd (EAGLE design)
At the start: 100 x 100 mm, 75 parts, among them IC1 MCP2551, IC2 DS18B20, IC3 MAX481CSA, K1 615064243321, K2 61400826021, K3 61400826021, K4 615016240521

Commit message: so much...
Parts:
- added R29: 4k7, schlager_passiv:R0805
- C3, C4: value (none) -> 100n
- C5, C6, C7: value (none) -> 22p
- R10, R2, R3, R4, R6, R7, R8, R9: value (none) -> 4k7
- R28: value (none) -> 1m
- U$2: device SparkFun-Boards:ARDUINO_PRO_MINI -> debauer_modules:ARDUINO_PRO_MINI
- moved IC1 1.27 mm to (65.5, 76.3)
Connections:
- removed net N$17: U$2.3
- new net RESET: U$1.17, U$2.3
- net A6: now also U$2.27
- net A7: now also U$2.28
- net D9_1W: now also R29.1
- net GND: now also IC1.2
- net P5V: now also IC1.3, R29.2
- net RX: now also IC3.1; no longer IC3.4
- net SCL: now also U$2.26
- net SDA: now also U$2.25
- net TX: now also IC3.4; no longer IC3.1
Routing:
- net A6: track 37.8 -> 74.4 mm, vias 5 -> 1
- net RESET: track 0.00 -> 33.4 mm, vias 0 -> 3
- net SDA: track 34.6 -> 62.2 mm, vias 1 -> 3
- net P5V: track 217.5 -> 241.8 mm, vias 8 -> 10
- net SCL: track 36.7 -> 60.6 mm, vias 3 -> 4
- net RX: track 49.5 -> 60.1 mm, vias 1 -> 3
- net A7: track 35.0 -> 45.2 mm
- net CANH1: track 211.8 -> 221.8 mm
- net A1: track 42.3 -> 37.4 mm, vias 2 -> 4
- net TX: track 48.8 -> 51.2 mm
- net D9_1W: track 42.5 -> 44.3 mm
- net GND: track 134.3 -> 135.8 mm, vias 20 -> 21
- net ANALOG_V24: track 20.7 -> 22.1 mm
- net CANTX: track 29.0 -> 27.7 mm
- net CANH: track 14.4 -> 15.7 mm
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