File: Nodes Gen2/Power-hub/power.sch (EAGLE design)
At the start: 75 parts, among them IC1 MCP2551, IC2 DS18B20, IC3 MAX481CSA, K1 615064243321, K2 61400826021, K3 61400826021, K4 615016240521

Commit message: so much...
Parts:
- added R29: 4k7, schlager_passiv:R-EU_R0805
- C3, C4: value (none) -> 100n
- C5, C6, C7: value (none) -> 22p
- R10, R2, R3, R4, R6, R7, R8, R9: value (none) -> 4k7
- R28: value (none) -> 1m
- U$2: device SparkFun-Boards:ARDUINO_PRO_MINI -> debauer_modules:ARDUINO_PRO_MINI
Connections:
- removed net N$17: U$2.RST
- new net RESET: U$1.~RESET, U$2.RST
- net D9_1W: now also R29.1
- net GND: now also IC1G$2.GND
- net P5V: now also IC1G$2.VCC, R29.2
- net RX: now also IC3G$1.RO; no longer IC3G$1.DI
- net TX: now also IC3G$1.DI; no longer IC3G$1.RO
