File: Nodes Gen2/rpi_can_multi/rpi_can.brd (EAGLE design)
At the start: 66 x 55.9 mm, 37 parts, among them IC1 DS1820TO92, IC2 MCP2551, IC3 MAX481CSA, IC4 MCP2551, K4 615016240521

Commit message: so much...
Parts:
- added J2: (no value), Wuerth_TERMINAL_BLOCKS_rev16a:691322310003
- added JP4: (no value), pinhead:1X03
- moved IC1 23.4 mm to (34.3, 33.2)
- moved R1 23.4 mm to (34.1, 38.3)
- moved C4 6.35 mm to (44.5, 30.2)
- moved C9 6.35 mm to (38.7, 45.7)
- moved IC4 6.35 mm to (47.0, 27.9)
- moved JP1 6.35 mm to (40.6, 24.1)
- moved R10 6.35 mm to (42.2, 45.7)
- moved R4 6.35 mm to (48.4, 25.4)
- moved R5 6.35 mm to (40.6, 30.3)
- moved R8 6.35 mm to (40.6, 27.9)
- moved U$1 6.35 mm to (47.0, 38.1)
- moved R12 6.35 mm to (37.9, 24.1)
- moved C2 5.08 mm to (43.2, 14.0)
- moved C3 5.08 mm to (48.3, 14.0)
- moved Q2 5.08 mm to (45.7, 17.8)
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Connections:
- net GND: now also J2.2, JP4.2
- net RS485_A: now also J2.1, JP4.1
- net RS485_B: now also J2.3, JP4.3
Routing:
- net RS485_A: track 23.3 -> 86.3 mm, vias 4 -> 6
- net RS485_B: track 20.8 -> 72.2 mm, vias 2 -> 4
- net 1W: track 49.6 -> 33.4 mm
- net CANH2: track 70.1 -> 75.9 mm
- net INT1: track 19.3 -> 24.8 mm
- net CANL2: track 76.0 -> 81.2 mm
- net SCK: track 21.1 -> 16.0 mm
- net CANL1: track 73.8 -> 76.4 mm
- net P5V: track 80.5 -> 83.0 mm
- net CANH1: track 88.7 -> 90.7 mm
- net MCP_OSC2: track 22.4 -> 24.2 mm
- net MCP_OSC1: track 27.8 -> 29.6 mm
- net CS1: track 15.6 -> 13.9 mm, vias 2 -> 0
- net MISO: track 38.5 -> 39.8 mm
- net MOSI: track 41.1 -> 42.3 mm
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Other:
- board text added: "A"
- board text added: "B"
- board text added: "G"
- board text added: "H"
- board text added: "L"
- board text added: "V"
- board text removed: "24V"
- board text removed: "GND"
